File: sensor_board.sch (KiCad schematic (older format))
At the start: 13 parts, among them P1 CONN_01X06, P2 CONN_01X10

Commit message: Cleaned up schematics and sensor board PCB
Parts:
- removed LED1, LED2: WS2812B, custom:PLCC4-5050, symbol WS2812B
- removed P2: CONN_01X10, Pin_Headers:Pin_Header_Angled_1x10, symbol CONN_01X10
- added J1: HEADER_5x2, Socket_Strips:Socket_Strip_Straight_2x05, symbol HEADER_5x2
- added J2: HEADER_2, Socket_Strips:Socket_Strip_Straight_1x02, symbol HEADER_2
- R2, R4, R6: value 100k -> 1M; footprint Resistors_Universal:Resistor_SMD+THTuniversal_0805to1206_RM10_HandSoldering_RevA_Date25Jun2010 -> Resistors_ThroughHole:Resistor_Horizontal_RM10mm
- R8: renamed from R9; value 100k -> 1M; footprint Resistors_Universal:Resistor_SMD+THTuniversal_0805to1206_RM10_HandSoldering_RevA_Date25Jun2010 -> Resistors_ThroughHole:Resistor_Horizontal_RM10mm
- renumbered R8 to R7, R7 to R9
Connections:
- net labels added: BUZZER
- net labels removed: +5V, NEOPIXEL_IN
- wire segments 53 -> 43
- no-connect marks 1 -> 2
Other:
- note added: "Flex sensor dividers"
- note added: "Interboard communication header"
- note added: "Optional buzzer"
- note added: "Pololu AltIMU-10 header"
- moved on the sheet: P1, R1, R2, R3, R4, R5, R6, R7, R8, R9

Commit message: Sensor board revised fit within a 5cmX5cm square
Parts:
- added D1: LED, w_smd_leds:Led_0805, symbol LED
- added R10: 1k, Resistors_SMD:R_0805_HandSoldering, symbol R
Connections:
- net +3V3: now also D1.2 (A)
- net GND: now also R10.1
- net VIN: now reaches P1.4 (P4)
- net VIN: now also J1.10
- new net: D1.1 (K), R10.2
- no-connect marks 2 -> 0
Changed lines of the file:
@@
 LIBS:w_transistor
 LIBS:w_vacuum
+LIBS:sensor_board-cache
 EELAYER 25 0
 EELAYER END
@@
 $EndComp
 $Comp
-L +3.3V #PWR01
+L +3.3V #PWR3
 U 1 1 56BFFEBE
 P 4550 3150
-F 0 "#PWR01" H 4550 3000 50  0001 C CNN
+F 0 "#PWR3" H 4550 3000 50  0001 C CNN
 F 1 "+3.3V" H 4550 3290 50  0000 C CNN
 F 2 "" H 4550 3150 50  0000 C CNN
@@
 $EndComp
 $Comp
-L GND #PWR02
+L GND #PWR4
 U 1 1 56C001EB
 P 4550 4900
-F 0 "#PWR02" H 4550 4650 50  0001 C CNN
+F 0 "#PWR4" H 4550 4650 50  0001 C CNN
 F 1 "GND" H 4550 4750 50  0000 C CNN
 F 2 "" H 4550 4900 50  0000 C CNN
@@
 SCL\nSDA\nGND\nVIN\nVDD\nSA0
 $Comp
-L GND #PWR03
+L GND #PWR5
 U 1 1 56C01386
 P 7150 4300
-F 0 "#PWR03" H 7150 4050 50  0001 C CNN
+F 0 "#PWR5" H 7150 4050 50  0001 C CNN
 F 1 "GND" H 7150 4150 50  0000 C CNN
 F 2 "" H 7150 4300 50  0000 C CNN
@@
 $EndComp
 $Comp
-L +3.3V #PWR04
+L +3.3V #PWR6
 U 1 1 56C014A7
 P 7250 3600
-F 0 "#PWR04" H 7250 3450 50  0001 C CNN
+F 0 "#PWR6" H 7250 3450 50  0001 C CNN
 F 1 "+3.3V" H 7250 3740 50  0000 C CNN
 F 2 "" H 7250 3600 50  0000 C CNN
@@
 	0    1    1    0
 $EndComp
-NoConn ~ 7050 4000
 Text Label 7750 3700 2    60   ~ 0
 IMU_SCL
@@
 IMU_SDA
 $Comp
-L GND #PWR05
+L GND #PWR7
 U 1 1 56C0210D
 P 7700 4300
-F 0 "#PWR05" H 7700 4050 50  0001 C CNN
+F 0 "#PWR7" H 7700 4050 50  0001 C CNN
 F 1 "GND" H 7700 4150 50  0000 C CNN
 F 2 "" H 7700 4300 50  0000 C CNN
@@
 $EndComp
 $Comp
-L GND #PWR06
+L GND #PWR2
 U 1 1 56C04BC2
-P 2950 4250
-F 0 "#PWR06" H 2950 4000 50  0001 C CNN
-F 1 "GND" H 2950 4100 50  0000 C CNN
-F 2 "" H 2950 4250 50  0000 C CNN
-F 3 "" H 2950 4250 50  0000 C CNN
-	1    2950 4250
+P 3550 4700
+F 0 "#PWR2" H 3550 4450 50  0001 C CNN
+F 1 "GND" H 3550 4550 50  0000 C CNN
+F 2 "" H 3550 4700 50  0000 C CNN
+F 3 "" H 3550 4700 50  0000 C CNN
+	1    3550 4700
 	-1   0    0    -1
 $EndComp
@@
 Text Label 3350 3900 2    60   ~ 0
 IMU_SDA
-NoConn ~ 2800 4100
-$Comp
-L +3.3V #PWR07
+$Comp
+L +3.3V #PWR1
 U 1 1 56EFEABD
 P 2950 3550
-F 0 "#PWR07" H 2950 3400 50  0001 C CNN
+F 0 "#PWR1" H 2950 3400 50  0001 C CNN
 F 1 "+3.3V" H 2950 3690 50  0000 C CNN
 F 2 "" H 2950 3550 50  0000 C CNN
@@
 BUZZER
 $Comp
-L GND #PWR08
+L GND #PWR8
 U 1 1 56F0259C
 P 8900 4150
-F 0 "#PWR08" H 8900 3900 50  0001 C CNN
+F 0 "#PWR8" H 8900 3900 50  0001 C CNN
 F 1 "GND" H 8900 4000 50  0000 C CNN
 F 2 "" H 8900 4150 50  0000 C CNN
@@
 Text Notes 5000 2800 2    60   ~ 0
 Flex sensor dividers
-Text Notes 3350 3150 2    60   ~ 0
+Text Notes 3600 3250 2    60   ~ 0
 Interboard communication header
-Text Notes 7600 3250 2    60   ~ 0
+Text Notes 7800 3250 2    60   ~ 0
 Pololu AltIMU-10 header
-Text Notes 9050 3600 2    60   ~ 0
+Text Notes 9150 3600 2    60   ~ 0
 Optional buzzer
 Wire Wire Line
@@
 	2800 4000 2950 4000
 Wire Wire Line
-	2950 4000 2950 4250
-Wire Wire Line
-	2800 3700 2950 3700
+	2950 4000 2950 4650
+Wire Wire Line
+	2800 3700 3550 3700
 Wire Wire Line
 	2950 3700 2950 3550
@@
 Wire Wire Line
 	8900 4000 8900 4150
+Wire Wire Line
+	2800 4100 3350 4100
+Text Label 3350 4100 2    60   ~ 0
+VIN
+Text Label 7750 4000 2    60   ~ 0
+VIN
+Wire Wire Line
+	7050 4000 7750 4000
+$Comp
+L LED D1
+U 1 1 56F271D5
+P 3550 4000
+F 0 "D1" H 3550 4100 50  0000 C CNN
+F 1 "LED" H 3550 3900 50  0000 C CNN
+F 2 "w_smd_leds:Led_0805" H 3550 4000 50  0001 C CNN
+F 3 "" H 3550 4000 50  0000 C CNN
+	1    3550 4000
+	0    -1   -1   0
+$EndComp
+Wire Wire Line
+	3550 3700 3550 3800
+Connection ~ 2950 3700
+$Comp
+L R R10
+U 1 1 56F27C3E
+P 3550 4450
+F 0 "R10" V 3630 4450 50  0000 C CNN
+F 1 "1k" V 3550 4450 50  0000 C CNN
+F 2 "Resistors_SMD:R_0805_HandSoldering" V 3480 4450 50  0001 C CNN
+F 3 "" H 3550 4450 50  0000 C CNN
+	1    3550 4450
+	-1   0    0    1
+$EndComp
+Wire Wire Line
+	3550 4300 3550 4200
+Wire Wire Line
+	3550 4700 3550 4600
+Wire Wire Line
+	2950 4650 3550 4650
+Connection ~ 3550 4650
 $EndSCHEMATC

Commit message: Rearranged sensor board components for cleanliness
Other:
- note added: "Optional buzzer\n(PWM)"
- note removed: "Optional buzzer"
Changed lines of the file:
@@
 LIBS:contrib
 LIBS:valves
-LIBS:coincell
 LIBS:ftdi
-LIBS:gatedrivers
-LIBS:moar-connectors
-LIBS:moar-electromechanical
-LIBS:moar-infineon
-LIBS:moar-linear
-LIBS:moar-micrel
-LIBS:moar-microchip
-LIBS:moar-passives
-LIBS:MOAR-POWER
-LIBS:moar-texas
-LIBS:mounting-hole
 LIBS:onsemi
-LIBS:samtec
-LIBS:moar-displays
-LIBS:w_analog
-LIBS:w_connectors
-LIBS:w_device
-LIBS:w_logic
-LIBS:w_memory
-LIBS:w_microcontrollers
-LIBS:w_opto
-LIBS:w_relay
-LIBS:w_rtx
-LIBS:w_transistor
-LIBS:w_vacuum
 LIBS:sensor_board-cache
 EELAYER 25 0
@@
 Text Notes 7800 3250 2    60   ~ 0
 Pololu AltIMU-10 header
-Text Notes 9150 3600 2    60   ~ 0
-Optional buzzer
+Text Notes 8450 3600 0    60   ~ 0
+Optional buzzer\n(PWM)
 Wire Wire Line
 	4550 3250 4550 3150
